File: Hardware/MOSFET_Power_Switch.sch (EAGLE design)
At the start: 31 parts, among them J3 5.5x2.1mm Barrel, Q1 600mA/40V, Q2 100A/100V/6.8mΩ, U1 LMR14203

Commit message: Update power jack
Other:
- note added: "High Voltage Control"
- note removed: "Solenoid Control"
Changed lines of the file:
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@@
 <layer number="154" name="FabDoc2" color="7" fill="1" visible="yes" active="yes"/>
 <layer number="155" name="FabDoc3" color="7" fill="1" visible="yes" active="yes"/>
+<layer number="156" name="gesam-Maß" color="7" fill="1" visible="no" active="no"/>
+<layer number="157" name="FaceMchng" color="7" fill="1" visible="no" active="no"/>
+<layer number="158" name="FaceMMeas" color="7" fill="1" visible="no" active="no"/>
+<layer number="159" name="Geh-Bear2" color="7" fill="1" visible="no" active="no"/>
+<layer number="160" name="Topologie" color="7" fill="1" visible="no" active="no"/>
+<layer number="161" name="tomplace2" color="7" fill="1" visible="no" active="no"/>
 <layer number="166" name="AntennaArea" color="7" fill="1" visible="no" active="no"/>
 <layer number="168" name="4mmHeightArea" color="7" fill="1" visible="no" active="no"/>
@@
 <layer number="250" name="Descript" color="3" fill="1" visible="no" active="no"/>
 <layer number="251" name="SMDround" color="12" fill="11" visible="no" active="no"/>
+<layer number="252" name="BR-BS" color="7" fill="1" visible="no" active="no"/>
 <layer number="253" name="Extra" color="7" fill="1" visible="no" active="no"/>
 <layer number="254" name="cooling" color="7" fill="1" visible="yes" active="yes"/>
@@
 Off</text>
 <text x="93.98" y="101.6" size="2.54" layer="94" align="center">Valve/Solenoid</text>
-<text x="180.34" y="121.92" size="2.54" layer="94" align="center">Solenoid
+<text x="180.34" y="121.92" size="2.54" layer="94" align="center">High Voltage
 Control</text>
 <text x="88.9" y="175.26" size="2.54" layer="94" align="center">3.3V Buck</text>
@@
 which will not be processed correctly with this version.
 </note>
+<note version="8.3" severity="warning">
+Since Version 8.3, EAGLE supports URNs for individual library
+assets (packages, symbols, and devices). The URNs of those assets
+will not be understood (or retained) with this version.
+</note>
 </compatibility>
